File: Channel.kicad_sch (KiCad schematic)
At the start: 23 parts, among them Q1 T2N7002AK,LM, Q2 DMP3099L, U1 INA219BxD

Commit message: Fixed review comments
Parts:
- removed Q1: T2N7002AK,LM, Package_TO_SOT_SMD:SOT-23, symbol Simulation_SPICE:NMOS
- removed Q2: DMP3099L, Package_TO_SOT_SMD:SOT-23, symbol Simulation_SPICE:PMOS
- added U10: T2N7002AK,LM, Package_TO_SOT_SMD:SOT-23, symbol HeatingBoard:NMOS_Project
- added U6: DMP3099L, Package_TO_SOT_SMD:SOT-23, symbol HeatingBoard:PMOS_project
Connections:
- net GND: now also U10.2
- net VOUT: now also U6.3
- net at C2.1, R7.2, R8.1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: now also U10.1
- net at R10.1, R11.2, R12.1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: now also U6.2
- net at R13.2: now also U10.3
- net at R12.2, R13.1: now also U6.1
