File: HeatingBoard.kicad_sch (KiCad schematic)
At the start: 7 parts, among them J1 XT60, J2 Conn_01x05, J3 Conn_01x03, J4 Conn_01x06, J5 Conn_01x03

Commit message: Finished PCB
Parts:
- removed J1: XT60, HeatingBoard:AMASS_XT60-M, symbol HeatingBoard:XT60
- added C13, C14: 10u, Capacitor_SMD:C_0805_2012Metric_Pad1.18x1.45mm_HandSolder, symbol Device:C_Small
- added H1, H2, H3, H4: MountingHole_Pad, MountingHole:MountingHole_3.2mm_M3_Pad, symbol Mechanical:MountingHole_Pad
- added J1: Conn_01x02, HeatingBoard:PHOENIX_1935161, symbol Connector_Generic:Conn_01x02
- added TP1: TestPoint, TestPoint:TestPoint_Plated_Hole_D5.0mm, symbol Connector:TestPoint
- added U5: AZ1117-3.3, Package_TO_SOT_THT:TO-220-3_Vertical, symbol Regulator_Linear:AZ1117-3.3
- J2: renamed from J4; footprint (none) -> HeatingBoard:PHOENIX_1935200
- J3: renamed from J5; footprint (none) -> HeatingBoard:PHOENIX_1935174
- J4: renamed from J3; footprint (none) -> HeatingBoard:PHOENIX_1935174
- J5: renamed from J2; footprint (none) -> HeatingBoard:PHOENIX_1935190
- R1: renamed from R7; footprint (none) -> Resistor_SMD:R_0603_1608Metric_Pad0.98x0.95mm_HandSolder
- R2: renamed from R6; footprint (none) -> Resistor_SMD:R_0603_1608Metric_Pad0.98x0.95mm_HandSolder
Connections:
- net +3V3: now also C14.1, U5.2 (VO)
- net GND: now also J5.1 (Pin_1), C13.2, C14.2, J1.2 (Pin_2), TP1.1, U5.1 (GND); no longer J5.5 (Pin_5)
- net VBATT: now also C13.1, J1.1 (Pin_1), U5.3 (VI)
- net VOUT1: now also J5.5 (Pin_5); no longer J5.1 (Pin_1)
- net VOUT2: now also J5.4 (Pin_4); no longer J5.2 (Pin_2)
- net VOUT4: now also J5.2 (Pin_2); no longer J5.4 (Pin_4)
- no-connect marks 0 -> 4
Other:
- note added: "BACKUP REGULATOR (DNP)"
