File: HeatingBoard.kicad_sch (KiCad schematic)
At the start: 16 parts, among them J1 Conn_01x02, J2 Conn_01x06, J3 Conn_01x03, J4 Conn_01x03, J5 Conn_01x05, U5 AZ1117-3.3

Commit message: Fixed review comments
Parts:
- H5: footprint (none) -> HeatingBoard:QRcode
Changed lines of the file:
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@@
 	(text "BACKUP REGULATOR (DNP)\n"
 		(exclude_from_sim no)
-		(at 254 135.89 0)
+		(at 254 127 0)
 		(effects
 			(font
@@
 				(size 1.27 1.27)
 			)
+		)
+	)
+	(text_box "This regulator is not needed. Will only be placed in case this board needs to be self-sufficient."
+		(exclude_from_sim no)
+		(at 241.3 128.27 0)
+		(size 40.64 7.62)
+		(margins 0.9525 0.9525 0.9525 0.9525)
+		(stroke
+			(width 0)
+			(type dash)
+		)
+		(fill
+			(type none)
+		)
+		(effects
+			(font
+				(size 1.27 1.27)
+			)
+			(justify left top)
 		)
 	)
@@
 			)
 		)
-		(property "Footprint" ""
+		(property "Footprint" "HeatingBoard:QRcode"
 			(at 151.13 173.99 0)
 			(effects
