File: _autosave-HeatingBoard.kicad_sch (KiCad schematic)
At the start: 16 parts, among them J1 Conn_01x02, J2 Conn_01x06, J3 Conn_01x03, J4 Conn_01x03, J5 Conn_01x05, U5 AZ1117-3.3

Commit message: Added QR code and images
Parts:
- H5: footprint (none) -> HeatingBoard:QRcode
Changed lines of the file:
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@@
 			)
 		)
-		(property "Footprint" ""
+		(property "Footprint" "HeatingBoard:QRcode"
 			(at 151.13 173.99 0)
 			(effects
